File: PCB/MinecraftPad.kicad_pcb (KiCad board)
At the start: 2 copper layers, 100 x 86 mm, 45 parts, among them SW1 SW_Push, SW10 SW_Push, SW11 SW_Push, SW12 SW_Push, SW13 SW_Push, SW14 SW_Push, SW15 SW_Push, SW16 SW_Push, SW17 SW_Push, SW18 SW_Push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

Commit message: improvements
Parts:
- removed the H1 at (-501.5, -68.0)
- removed H3, H4: MountingHole, MountingHole:MountingHole_3.2mm_M3
- D1, D10, D11, D12, D13, D14, D15, D16, D17, D18, D19, D2, D20, D3, D4, D5, D6, D7, D8, D9: footprint Diode_SMD:D_1206_3216Metric -> Diode_SMD:D_0805_2012Metric_Pad1.15x1.40mm_HandSolder
- renumbered H2 to H1
Connections:
- B1 pad 13: Row3 -> Col1
- B1 pad 14: Row2 -> Col2
- B1 pad 15: Row1 -> Col3
- B1 pad 16: Col5 -> Row3
- B1 pad 17: Col4 -> Row2
- B1 pad 18: Col3 -> Row1
- B1 pad 19: Col2 -> Col5
- B1 pad 20: Col1 -> Col4
Routing:
- net Col1: track 0.00 -> 181.0 mm
- net Col2: track 0.00 -> 164.2 mm
- net Row4: track 0.00 -> 136.0 mm
- net Col3: track 0.00 -> 132.9 mm
- net Row3: track 0.00 -> 128.9 mm
- net Row2: track 0.00 -> 123.1 mm
- net Row1: track 0.00 -> 90.5 mm
- net Col5: track 0.00 -> 75.0 mm
- net Col4: track 0.00 -> 73.6 mm
- net GND: track 0.00 -> 18.8 mm
- net Net-(D20-Pad2): track 0.00 -> 9.39 mm
- net Net-(D1-Pad2): track 0.00 -> 8.90 mm
- net Net-(D9-Pad2): track 0.00 -> 8.69 mm
- net Net-(D8-Pad2): track 0.00 -> 8.69 mm
- net Net-(D7-Pad2): track 0.00 -> 8.69 mm
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- added copper zone on F.Cu, net (none)
Other:
- board text added: "CraftPad V0.1"

Commit message: v0.2
Parts:
- added Reset1: SW_Push, Button_Switch_THT:SW_PUSH_6mm, F.Cu at (-407.0, -61.0)
- D1, D10, D11, D12, D13, D14, D15, D16, D17, D18, D19, D2, D20, D3, D4, D5, D6, D7, D8, D9: footprint Diode_SMD:D_0805_2012Metric_Pad1.15x1.40mm_HandSolder -> Diode_SMD:D_0603_1608Metric_Pad1.05x0.95mm_HandSolder
Connections:
- B1 pad 22: (no net) -> Net-(B1-Pad22)
Routing:
- net Net-(B1-Pad22): track 0.00 -> 74.6 mm
- net GND: track 18.8 -> 90.9 mm
- net Row3: track 128.9 -> 127.6 mm
- added copper zone on F.Cu, net GND
- removed copper zone on F.Cu, net (none)
Other:
- board text added: "CraftPad V0.2"
- board text removed: "CraftPad V0.1"

Commit message: v0.2
Parts:
- added D21: LED_RGBC, LED_THT:LED_D5.0mm-4_RGB, B.Cu at (-499.0, -57.0)
- added R1: 220Ω, Resistor_THT:R_Axial_DIN0207_L6.3mm_D2.5mm_P10.16mm_Horizontal, F.Cu at (-498.0, -25.0)
- added R2: 220Ω, Resistor_THT:R_Axial_DIN0207_L6.3mm_D2.5mm_P10.16mm_Horizontal, F.Cu at (-498.0, -40.0)
- added R3: 220Ω, Resistor_THT:R_Axial_DIN0207_L6.3mm_D2.5mm_P10.16mm_Horizontal, F.Cu at (-498.0, -10.0)
Connections:
- B1 pad 10: (no net) -> Col1
- B1 pad 11: (no net) -> Row4
- B1 pad 12: Row4 -> Red
- B1 pad 13: Col1 -> (no net)
- B1 pad 8: (no net) -> Blue
- B1 pad 9: (no net) -> Green
Routing:
- net Blue: track 0.00 -> 38.4 mm
- net Net-(D21-Pad3): track 0.00 -> 37.5 mm
- net Net-(D21-Pad1): track 0.00 -> 22.4 mm
- net Col1: track 181.0 -> 199.5 mm
- net Red: track 0.00 -> 13.3 mm
- net Net-(D21-Pad2): track 0.00 -> 6.95 mm
- net Green: track 0.00 -> 6.89 mm
- net Row4: track 136.0 -> 139.7 mm
- net Col5: track 75.0 -> 74.5 mm
Other:
- board size 100 x 86 mm -> 103 x 86 mm

Commit message: v0.4
Connections:
- B1 pad 10: Col1 -> Row3
- B1 pad 14: Col2 -> Col5
- B1 pad 15: Col3 -> Col4
- B1 pad 16: Row3 -> Col3
- B1 pad 17: Row2 -> Col2
- B1 pad 18: Row1 -> Col1
- B1 pad 19: Col5 -> (no net)
- B1 pad 20: Col4 -> (no net)
- B1 pad 5: (no net) -> Row1
- B1 pad 7: (no net) -> Row2
Routing:
- net Col1: track 199.5 -> 136.7 mm
- net Col2: track 164.2 -> 114.2 mm
- net Col3: track 132.9 -> 91.7 mm
- net Row1: track 90.6 -> 100.5 mm
- net Row2: track 123.1 -> 116.6 mm
- net Row3: track 127.6 -> 131.8 mm
- net Col4: track 73.6 -> 71.4 mm
- net Row4: track 139.7 -> 138.1 mm
- net Col5: track 74.5 -> 73.9 mm

Commit message: update silkscreen
Other:
- board text added: "CraftPad V0.4 2021-04-05 James Sa"
- board text removed: "CraftPad V0.2"
Changed lines of the file:
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@@
   )
   (gr_arc (start -445 18) (end -439 18) (angle -180) (layer Edge.Cuts) (width 0.05))
-  (gr_text "CraftPad V0.2" (at -485 -20) (layer F.SilkS)
+  (gr_text "CraftPad V0.4\n2021-04-05\nJames Sa" (at -458.75 -62.75) (layer F.SilkS)
     (effects (font (size 1.5 1.5) (thickness 0.3)))
   )

Commit message: RGBA
Parts:
- D21: value LED_RGBC -> LED_RGBA; moved to F.Cu
- moved D21 1.06 mm to (-499.8, -56.2)
Connections:
- B1 pad 21: (no net) -> VCC
- D21 pad 4: GND -> VCC
Routing:
- net VCC: track 0.00 -> 20.1 mm
- net Net-(D21-Pad2): track 6.95 -> 6.29 mm
- net Net-(D21-Pad1): track 22.4 -> 21.8 mm

Commit message: v0.5
Parts:
- removed H1: MountingHole, MountingHole:MountingHole_3.2mm_M3
- D21: value LED_RGBA -> LED_RCGB; moved to B.Cu
- R1, R2, R3: moved to B.Cu
- moved R1 15.0 mm to (-497.8, -40.0), turned to 270 degrees
- moved R2 14.1 mm to (-497.8, -25.9), turned to 270 degrees
- moved D21 6.25 mm to (-499.6, -50.0)
- moved R3 1.77 mm to (-497.8, -11.8), turned to 270 degrees
Connections:
- B1 pad 21: VCC -> (no net)
- D21 pad 2: Net-(D21-Pad2) -> GND
- D21 pad 4: VCC -> Net-(D21-Pad4)
- R1 pad 1: Red -> Blue
- R1 pad 2: Net-(D21-Pad1) -> Net-(D21-Pad4)
- R2 pad 2: Net-(D21-Pad2) -> Net-(D21-Pad3)
- R3 pad 1: Blue -> Red
- R3 pad 2: Net-(D21-Pad3) -> Net-(D21-Pad1)
Routing:
- net Blue: track 38.4 -> 8.36 mm
- net Net-(D21-Pad1): track 21.8 -> 49.4 mm
- net Net-(D21-Pad4): track 0.00 -> 21.5 mm
- net VCC: track 20.1 -> 0.00 mm
- net Red: track 13.3 -> 26.4 mm
- net Green: track 6.89 -> 19.9 mm
- net Net-(D21-Pad2): track 6.29 -> 0.00 mm
- net Row4: track 138.1 -> 137.2 mm
- net Net-(D21-Pad3): track 37.2 -> 36.6 mm
Other:
- board text added: "CraftPad V0.5 2021-04-06 James Sa"
- board text removed: "CraftPad V0.4 2021-04-05 James Sa"
