File: PCB/MinecraftPad.sch (KiCad schematic (older format))
At the start: 45 parts, among them SW1 SW_Push, SW10 SW_Push, SW11 SW_Push, SW12 SW_Push, SW13 SW_Push, SW14 SW_Push, SW15 SW_Push, SW16 SW_Push, SW17 SW_Push, SW18 SW_Push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

Commit message: improvements
Parts:
- removed H1, H3, H4: MountingHole, MountingHole:MountingHole_3.2mm_M3, symbol Mechanical:MountingHole
- D1, D10, D11, D12, D13, D14, D15, D16, D17, D18, D19, D2, D20, D3, D4, D5, D6, D7, D8, D9: footprint Diode_SMD:D_1206_3216Metric -> Diode_SMD:D_0805_2012Metric_Pad1.15x1.40mm_HandSolder
- renumbered H2 to H1
Changed lines of the file:
@@
 $EndDescr
-$Comp
-L SparkFun-Boards:SPARKFUN_PRO_MICRO B1
-U 1 1 6065E65E
-P 2800 2300
-F 0 "B1" H 2800 3210 45  0000 C CNN
-F 1 "PRO MICRO" H 2800 3126 45  0000 C CNN
-F 2 "footprints:ArduinoProMicro" H 2800 3100 20  0001 C CNN
-F 3 "" H 2800 2300 50  0001 C CNN
-F 4 "XXX-00000" H 2800 3031 60  0001 C CNN "Field4"
-	1    2800 2300
-	1    0    0    -1
-$EndComp
 $Comp
 L power:PWR_FLAG #FLG02
@@
 F 0 "D1" V 4096 3770 50  0000 R CNN
 F 1 "D" V 4005 3770 50  0000 R CNN
-F 2 "Diode_SMD:D_1206_3216Metric" H 4050 3850 50  0001 C CNN
+F 2 "Diode_SMD:D_0805_2012Metric_Pad1.15x1.40mm_HandSolder" H 4050 3850 50  0001 C CNN
 F 3 "~" H 4050 3850 50  0001 C CNN
 	1    4050 3850
@@
 F 0 "D6" V 4096 4470 50  0000 R CNN
 F 1 "D" V 4005 4470 50  0000 R CNN
-F 2 "Diode_SMD:D_1206_3216Metric" H 4050 4550 50  0001 C CNN
+F 2 "Diode_SMD:D_0805_2012Metric_Pad1.15x1.40mm_HandSolder" H 4050 4550 50  0001 C CNN
 F 3 "~" H 4050 4550 50  0001 C CNN
 	1    4050 4550
@@
 F 0 "D11" V 4096 5220 50  0000 R CNN
 F 1 "D" V 4005 5220 50  0000 R CNN
-F 2 "Diode_SMD:D_1206_3216Metric" H 4050 5300 50  0001 C CNN
+F 2 "Diode_SMD:D_0805_2012Metric_Pad1.15x1.40mm_HandSolder" H 4050 5300 50  0001 C CNN
 F 3 "~" H 4050 5300 50  0001 C CNN
 	1    4050 5300
@@
 F 0 "D16" V 4096 5970 50  0000 R CNN
 F 1 "D" V 4005 5970 50  0000 R CNN
-F 2 "Diode_SMD:D_1206_3216Metric" H 4050 6050 50  0001 C CNN
+F 2 "Diode_SMD:D_0805_2012Metric_Pad1.15x1.40mm_HandSolder" H 4050 6050 50  0001 C CNN
 F 3 "~" H 4050 6050 50  0001 C CNN
 	1    4050 6050
@@
 F 0 "D2" V 5296 3770 50  0000 R CNN
 F 1 "D" V 5205 3770 50  0000 R CNN
-F 2 "Diode_SMD:D_1206_3216Metric" H 5250 3850 50  0001 C CNN
+F 2 "Diode_SMD:D_0805_2012Metric_Pad1.15x1.40mm_HandSolder" H 5250 3850 50  0001 C CNN
 F 3 "~" H 5250 3850 50  0001 C CNN
 	1    5250 3850
@@
 F 0 "D7" V 5296 4470 50  0000 R CNN
 F 1 "D" V 5205 4470 50  0000 R CNN
-F 2 "Diode_SMD:D_1206_3216Metric" H 5250 4550 50  0001 C CNN
+F 2 "Diode_SMD:D_0805_2012Metric_Pad1.15x1.40mm_HandSolder" H 5250 4550 50  0001 C CNN
 F 3 "~" H 5250 4550 50  0001 C CNN
 	1    5250 4550
@@
 F 0 "D12" V 5296 5220 50  0000 R CNN
 F 1 "D" V 5205 5220 50  0000 R CNN
-F 2 "Diode_SMD:D_1206_3216Metric" H 5250 5300 50  0001 C CNN
+F 2 "Diode_SMD:D_0805_2012Metric_Pad1.15x1.40mm_HandSolder" H 5250 5300 50  0001 C CNN
 F 3 "~" H 5250 5300 50  0001 C CNN
 	1    5250 5300
@@
 F 0 "D17" V 5296 5970 50  0000 R CNN
 F 1 "D" V 5205 5970 50  0000 R CNN
-F 2 "Diode_SMD:D_1206_3216Metric" H 5250 6050 50  0001 C CNN
+F 2 "Diode_SMD:D_0805_2012Metric_Pad1.15x1.40mm_HandSolder" H 5250 6050 50  0001 C CNN
 F 3 "~" H 5250 6050 50  0001 C CNN
 	1    5250 6050
@@
 F 0 "D3" V 6496 3770 50  0000 R CNN
 F 1 "D" V 6405 3770 50  0000 R CNN
-F 2 "Diode_SMD:D_1206_3216Metric" H 6450 3850 50  0001 C CNN
+F 2 "Diode_SMD:D_0805_2012Metric_Pad1.15x1.40mm_HandSolder" H 6450 3850 50  0001 C CNN
 F 3 "~" H 6450 3850 50  0001 C CNN
 	1    6450 3850
@@
 F 0 "D8" V 6496 4470 50  0000 R CNN
 F 1 "D" V 6405 4470 50  0000 R CNN
-F 2 "Diode_SMD:D_1206_3216Metric" H 6450 4550 50  0001 C CNN
+F 2 "Diode_SMD:D_0805_2012Metric_Pad1.15x1.40mm_HandSolder" H 6450 4550 50  0001 C CNN
 F 3 "~" H 6450 4550 50  0001 C CNN
 	1    6450 4550
@@
 F 0 "D13" V 6496 5220 50  0000 R CNN
 F 1 "D" V 6405 5220 50  0000 R CNN
-F 2 "Diode_SMD:D_1206_3216Metric" H 6450 5300 50  0001 C CNN
+F 2 "Diode_SMD:D_0805_2012Metric_Pad1.15x1.40mm_HandSolder" H 6450 5300 50  0001 C CNN
 F 3 "~" H 6450 5300 50  0001 C CNN
 	1    6450 5300
@@
 F 0 "D18" V 6496 5970 50  0000 R CNN
 F 1 "D" V 6405 5970 50  0000 R CNN
-F 2 "Diode_SMD:D_1206_3216Metric" H 6450 6050 50  0001 C CNN
+F 2 "Diode_SMD:D_0805_2012Metric_Pad1.15x1.40mm_HandSolder" H 6450 6050 50  0001 C CNN
 F 3 "~" H 6450 6050 50  0001 C CNN
 	1    6450 6050
@@
 F 0 "D4" V 7696 3770 50  0000 R CNN
 F 1 "D" V 7605 3770 50  0000 R CNN
-F 2 "Diode_SMD:D_1206_3216Metric" H 7650 3850 50  0001 C CNN
+F 2 "Diode_SMD:D_0805_2012Metric_Pad1.15x1.40mm_HandSolder" H 7650 3850 50  0001 C CNN
 F 3 "~" H 7650 3850 50  0001 C CNN
 	1    7650 3850
@@
 F 0 "D9" V 7696 4470 50  0000 R CNN
 F 1 "D" V 7605 4470 50  0000 R CNN
-F 2 "Diode_SMD:D_1206_3216Metric" H 7650 4550 50  0001 C CNN
+F 2 "Diode_SMD:D_0805_2012Metric_Pad1.15x1.40mm_HandSolder" H 7650 4550 50  0001 C CNN
 F 3 "~" H 7650 4550 50  0001 C CNN
 	1    7650 4550
@@
 F 0 "D14" V 7696 5220 50  0000 R CNN
 F 1 "D" V 7605 5220 50  0000 R CNN
-F 2 "Diode_SMD:D_1206_3216Metric" H 7650 5300 50  0001 C CNN
+F 2 "Diode_SMD:D_0805_2012Metric_Pad1.15x1.40mm_HandSolder" H 7650 5300 50  0001 C CNN
 F 3 "~" H 7650 5300 50  0001 C CNN
 	1    7650 5300
@@
 F 0 "D19" V 7696 5970 50  0000 R CNN
 F 1 "D" V 7605 5970 50  0000 R CNN
-F 2 "Diode_SMD:D_1206_3216Metric" H 7650 6050 50  0001 C CNN
+F 2 "Diode_SMD:D_0805_2012Metric_Pad1.15x1.40mm_HandSolder" H 7650 6050 50  0001 C CNN
 F 3 "~" H 7650 6050 50  0001 C CNN
 	1    7650 6050
@@
 F 0 "D5" V 9196 3770 50  0000 R CNN
 F 1 "D" V 9105 3770 50  0000 R CNN
-F 2 "Diode_SMD:D_1206_3216Metric" H 9150 3850 50  0001 C CNN
+F 2 "Diode_SMD:D_0805_2012Metric_Pad1.15x1.40mm_HandSolder" H 9150 3850 50  0001 C CNN
 F 3 "~" H 9150 3850 50  0001 C CNN
 	1    9150 3850
@@
 F 0 "D10" V 9196 4470 50  0000 R CNN
 F 1 "D" V 9105 4470 50  0000 R CNN
-F 2 "Diode_SMD:D_1206_3216Metric" H 9150 4550 50  0001 C CNN
+F 2 "Diode_SMD:D_0805_2012Metric_Pad1.15x1.40mm_HandSolder" H 9150 4550 50  0001 C CNN
 F 3 "~" H 9150 4550 50  0001 C CNN
 	1    9150 4550
@@
 F 0 "D15" V 9196 5220 50  0000 R CNN
 F 1 "D" V 9105 5220 50  0000 R CNN
-F 2 "Diode_SMD:D_1206_3216Metric" H 9150 5300 50  0001 C CNN
+F 2 "Diode_SMD:D_0805_2012Metric_Pad1.15x1.40mm_HandSolder" H 9150 5300 50  0001 C CNN
 F 3 "~" H 9150 5300 50  0001 C CNN
 	1    9150 5300
@@
 F 0 "D20" V 9196 5970 50  0000 R CNN
 F 1 "D" V 9105 5970 50  0000 R CNN
-F 2 "Diode_SMD:D_1206_3216Metric" H 9150 6050 50  0001 C CNN
+F 2 "Diode_SMD:D_0805_2012Metric_Pad1.15x1.40mm_HandSolder" H 9150 6050 50  0001 C CNN
 F 3 "~" H 9150 6050 50  0001 C CNN
 	1    9150 6050
@@
 	2350 2050 1400 2050
 Connection ~ 1400 2050
-Text GLabel 3250 2150 2    50   Input ~ 0
+Text GLabel 3250 2850 2    50   Input ~ 0
 Col1
-Text GLabel 3250 2250 2    50   Input ~ 0
-Col2
 Text GLabel 3250 2350 2    50   Input ~ 0
-Col3
+Row1
 Text GLabel 3250 2450 2    50   Input ~ 0
-Col4
+Row2
 Text GLabel 3250 2550 2    50   Input ~ 0
-Col5
-Text GLabel 3250 2650 2    50   Input ~ 0
-Row1
-Text GLabel 3250 2750 2    50   Input ~ 0
-Row2
-Text GLabel 3250 2850 2    50   Input ~ 0
 Row3
 Text GLabel 2350 2850 0    50   Input ~ 0
@@
 $EndComp
 Wire Wire Line
-	3250 1850 3950 1850
-Wire Wire Line
 	3950 1850 3950 2050
 Wire Wire Line
 	3750 1650 3750 2050
-Wire Wire Line
-	3750 2050 3250 2050
 $Comp
 L Mechanical:MountingHole H1
-U 1 1 607BA992
-P 7100 1850
-F 0 "H1" H 7200 1896 50  0000 L CNN
-F 1 "MountingHole" H 7200 1805 50  0000 L CNN
-F 2 "MountingHole:MountingHole_3.2mm_M3" H 7100 1850 50  0001 C CNN
-F 3 "~" H 7100 1850 50  0001 C CNN
-	1    7100 1850
-	1    0    0    -1
-$EndComp
-$Comp
-L Mechanical:MountingHole H2
 U 1 1 607BB18A
 P 7550 1850
-F 0 "H2" H 7650 1896 50  0000 L CNN
+F 0 "H1" H 7650 1896 50  0000 L CNN
 F 1 "MountingHole" H 7650 1805 50  0000 L CNN
 F 2 "MountingHole:MountingHole_3.2mm_M3" H 7550 1850 50  0001 C CNN
@@
 	1    0    0    -1
 $EndComp
-$Comp
-L Mechanical:MountingHole H4
-U 1 1 607BBAB8
-P 7200 2150
-F 0 "H4" H 7300 2196 50  0000 L CNN
-F 1 "MountingHole" H 7300 2105 50  0000 L CNN
-F 2 "MountingHole:MountingHole_3.2mm_M3" H 7200 2150 50  0001 C CNN
-F 3 "~" H 7200 2150 50  0001 C CNN
-	1    7200 2150
-	1    0    0    -1
-$EndComp
-$Comp
-L Mechanical:MountingHole H3
-U 1 1 607BC1C0
-P 7600 2100
-F 0 "H3" H 7700 2146 50  0000 L CNN
-F 1 "MountingHole" H 7700 2055 50  0000 L CNN
-F 2 "MountingHole:MountingHole_3.2mm_M3" H 7600 2100 50  0001 C CNN
-F 3 "~" H 7600 2100 50  0001 C CNN
-	1    7600 2100
-	1    0    0    -1
-$EndComp
+Text GLabel 3250 2650 2    50   Input ~ 0
+Col3
+Text GLabel 3250 2750 2    50   Input ~ 0
+Col2
+Text GLabel 3250 2250 2    50   Input ~ 0
+Col5
+Wire Wire Line
+	3750 2050 3250 2050
+Wire Wire Line
+	3250 1850 3950 1850
+Text GLabel 3250 2150 2    50   Input ~ 0
+Col4
+$Comp
+L SparkFun-Boards:SPARKFUN_PRO_MICRO B1
+U 1 1 6065E65E
+P 2800 2300
+F 0 "B1" H 2800 3210 45  0000 C CNN
+F 1 "PRO MICRO" H 2800 3126 45  0000 C CNN
+F 2 "footprints:ArduinoProMicro" H 2800 3100 20  0001 C CNN
+F 3 "" H 2800 2300 50  0001 C CNN
+F 4 "XXX-00000" H 2800 3031 60  0001 C CNN "Field4"
+	1    2800 2300
+	1    0    0    -1
+$EndComp

Commit message: v0.2
Parts:
- added Reset1: SW_Push, Button_Switch_THT:SW_PUSH_6mm, symbol Switch:SW_Push
- D1, D10, D11, D12, D13, D14, D15, D16, D17, D18, D19, D2, D20, D3, D4, D5, D6, D7, D8, D9: footprint Diode_SMD:D_0805_2012Metric_Pad1.15x1.40mm_HandSolder -> Diode_SMD:D_0603_1608Metric_Pad1.05x0.95mm_HandSolder
Connections:
- wire segments 53 -> 56
- no-connect marks 11 -> 10
Changed lines of the file:
@@
 encoding utf-8
 Sheet 1 1
-Title ""
-Date ""
-Rev ""
-Comp ""
+Title "CraftPad"
+Date "2021-04-02"
+Rev "V0.2"
+Comp "James Sa"
 Comment1 ""
 Comment2 ""
@@
 F 0 "D1" V 4096 3770 50  0000 R CNN
 F 1 "D" V 4005 3770 50  0000 R CNN
-F 2 "Diode_SMD:D_0805_2012Metric_Pad1.15x1.40mm_HandSolder" H 4050 3850 50  0001 C CNN
+F 2 "Diode_SMD:D_0603_1608Metric_Pad1.05x0.95mm_HandSolder" H 4050 3850 50  0001 C CNN
 F 3 "~" H 4050 3850 50  0001 C CNN
 	1    4050 3850
@@
 F 0 "D6" V 4096 4470 50  0000 R CNN
 F 1 "D" V 4005 4470 50  0000 R CNN
-F 2 "Diode_SMD:D_0805_2012Metric_Pad1.15x1.40mm_HandSolder" H 4050 4550 50  0001 C CNN
+F 2 "Diode_SMD:D_0603_1608Metric_Pad1.05x0.95mm_HandSolder" H 4050 4550 50  0001 C CNN
 F 3 "~" H 4050 4550 50  0001 C CNN
 	1    4050 4550
@@
 F 0 "D11" V 4096 5220 50  0000 R CNN
 F 1 "D" V 4005 5220 50  0000 R CNN
-F 2 "Diode_SMD:D_0805_2012Metric_Pad1.15x1.40mm_HandSolder" H 4050 5300 50  0001 C CNN
+F 2 "Diode_SMD:D_0603_1608Metric_Pad1.05x0.95mm_HandSolder" H 4050 5300 50  0001 C CNN
 F 3 "~" H 4050 5300 50  0001 C CNN
 	1    4050 5300
@@
 F 0 "D16" V 4096 5970 50  0000 R CNN
 F 1 "D" V 4005 5970 50  0000 R CNN
-F 2 "Diode_SMD:D_0805_2012Metric_Pad1.15x1.40mm_HandSolder" H 4050 6050 50  0001 C CNN
+F 2 "Diode_SMD:D_0603_1608Metric_Pad1.05x0.95mm_HandSolder" H 4050 6050 50  0001 C CNN
 F 3 "~" H 4050 6050 50  0001 C CNN
 	1    4050 6050
@@
 F 0 "D2" V 5296 3770 50  0000 R CNN
 F 1 "D" V 5205 3770 50  0000 R CNN
-F 2 "Diode_SMD:D_0805_2012Metric_Pad1.15x1.40mm_HandSolder" H 5250 3850 50  0001 C CNN
+F 2 "Diode_SMD:D_0603_1608Metric_Pad1.05x0.95mm_HandSolder" H 5250 3850 50  0001 C CNN
 F 3 "~" H 5250 3850 50  0001 C CNN
 	1    5250 3850
@@
 F 0 "D7" V 5296 4470 50  0000 R CNN
 F 1 "D" V 5205 4470 50  0000 R CNN
-F 2 "Diode_SMD:D_0805_2012Metric_Pad1.15x1.40mm_HandSolder" H 5250 4550 50  0001 C CNN
+F 2 "Diode_SMD:D_0603_1608Metric_Pad1.05x0.95mm_HandSolder" H 5250 4550 50  0001 C CNN
 F 3 "~" H 5250 4550 50  0001 C CNN
 	1    5250 4550
@@
 F 0 "D12" V 5296 5220 50  0000 R CNN
 F 1 "D" V 5205 5220 50  0000 R CNN
-F 2 "Diode_SMD:D_0805_2012Metric_Pad1.15x1.40mm_HandSolder" H 5250 5300 50  0001 C CNN
+F 2 "Diode_SMD:D_0603_1608Metric_Pad1.05x0.95mm_HandSolder" H 5250 5300 50  0001 C CNN
 F 3 "~" H 5250 5300 50  0001 C CNN
 	1    5250 5300
@@
 F 0 "D17" V 5296 5970 50  0000 R CNN
 F 1 "D" V 5205 5970 50  0000 R CNN
-F 2 "Diode_SMD:D_0805_2012Metric_Pad1.15x1.40mm_HandSolder" H 5250 6050 50  0001 C CNN
+F 2 "Diode_SMD:D_0603_1608Metric_Pad1.05x0.95mm_HandSolder" H 5250 6050 50  0001 C CNN
 F 3 "~" H 5250 6050 50  0001 C CNN
 	1    5250 6050
@@
 F 0 "D3" V 6496 3770 50  0000 R CNN
 F 1 "D" V 6405 3770 50  0000 R CNN
-F 2 "Diode_SMD:D_0805_2012Metric_Pad1.15x1.40mm_HandSolder" H 6450 3850 50  0001 C CNN
+F 2 "Diode_SMD:D_0603_1608Metric_Pad1.05x0.95mm_HandSolder" H 6450 3850 50  0001 C CNN
 F 3 "~" H 6450 3850 50  0001 C CNN
 	1    6450 3850
@@
 F 0 "D8" V 6496 4470 50  0000 R CNN
 F 1 "D" V 6405 4470 50  0000 R CNN
-F 2 "Diode_SMD:D_0805_2012Metric_Pad1.15x1.40mm_HandSolder" H 6450 4550 50  0001 C CNN
+F 2 "Diode_SMD:D_0603_1608Metric_Pad1.05x0.95mm_HandSolder" H 6450 4550 50  0001 C CNN
 F 3 "~" H 6450 4550 50  0001 C CNN
 	1    6450 4550
@@
 F 0 "D13" V 6496 5220 50  0000 R CNN
 F 1 "D" V 6405 5220 50  0000 R CNN
-F 2 "Diode_SMD:D_0805_2012Metric_Pad1.15x1.40mm_HandSolder" H 6450 5300 50  0001 C CNN
+F 2 "Diode_SMD:D_0603_1608Metric_Pad1.05x0.95mm_HandSolder" H 6450 5300 50  0001 C CNN
 F 3 "~" H 6450 5300 50  0001 C CNN
 	1    6450 5300
@@
 F 0 "D18" V 6496 5970 50  0000 R CNN
 F 1 "D" V 6405 5970 50  0000 R CNN
-F 2 "Diode_SMD:D_0805_2012Metric_Pad1.15x1.40mm_HandSolder" H 6450 6050 50  0001 C CNN
+F 2 "Diode_SMD:D_0603_1608Metric_Pad1.05x0.95mm_HandSolder" H 6450 6050 50  0001 C CNN
 F 3 "~" H 6450 6050 50  0001 C CNN
 	1    6450 6050
@@
 F 0 "D4" V 7696 3770 50  0000 R CNN
 F 1 "D" V 7605 3770 50  0000 R CNN
-F 2 "Diode_SMD:D_0805_2012Metric_Pad1.15x1.40mm_HandSolder" H 7650 3850 50  0001 C CNN
+F 2 "Diode_SMD:D_0603_1608Metric_Pad1.05x0.95mm_HandSolder" H 7650 3850 50  0001 C CNN
 F 3 "~" H 7650 3850 50  0001 C CNN
 	1    7650 3850
@@
 F 0 "D9" V 7696 4470 50  0000 R CNN
 F 1 "D" V 7605 4470 50  0000 R CNN
-F 2 "Diode_SMD:D_0805_2012Metric_Pad1.15x1.40mm_HandSolder" H 7650 4550 50  0001 C CNN
+F 2 "Diode_SMD:D_0603_1608Metric_Pad1.05x0.95mm_HandSolder" H 7650 4550 50  0001 C CNN
 F 3 "~" H 7650 4550 50  0001 C CNN
 	1    7650 4550
@@
 F 0 "D14" V 7696 5220 50  0000 R CNN
 F 1 "D" V 7605 5220 50  0000 R CNN
-F 2 "Diode_SMD:D_0805_2012Metric_Pad1.15x1.40mm_HandSolder" H 7650 5300 50  0001 C CNN
+F 2 "Diode_SMD:D_0603_1608Metric_Pad1.05x0.95mm_HandSolder" H 7650 5300 50  0001 C CNN
 F 3 "~" H 7650 5300 50  0001 C CNN
 	1    7650 5300
@@
 F 0 "D19" V 7696 5970 50  0000 R CNN
 F 1 "D" V 7605 5970 50  0000 R CNN
-F 2 "Diode_SMD:D_0805_2012Metric_Pad1.15x1.40mm_HandSolder" H 7650 6050 50  0001 C CNN
+F 2 "Diode_SMD:D_0603_1608Metric_Pad1.05x0.95mm_HandSolder" H 7650 6050 50  0001 C CNN
 F 3 "~" H 7650 6050 50  0001 C CNN
 	1    7650 6050
@@
 F 0 "D5" V 9196 3770 50  0000 R CNN
 F 1 "D" V 9105 3770 50  0000 R CNN
-F 2 "Diode_SMD:D_0805_2012Metric_Pad1.15x1.40mm_HandSolder" H 9150 3850 50  0001 C CNN
+F 2 "Diode_SMD:D_0603_1608Metric_Pad1.05x0.95mm_HandSolder" H 9150 3850 50  0001 C CNN
 F 3 "~" H 9150 3850 50  0001 C CNN
 	1    9150 3850
@@
 F 0 "D10" V 9196 4470 50  0000 R CNN
 F 1 "D" V 9105 4470 50  0000 R CNN
-F 2 "Diode_SMD:D_0805_2012Metric_Pad1.15x1.40mm_HandSolder" H 9150 4550 50  0001 C CNN
+F 2 "Diode_SMD:D_0603_1608Metric_Pad1.05x0.95mm_HandSolder" H 9150 4550 50  0001 C CNN
 F 3 "~" H 9150 4550 50  0001 C CNN
 	1    9150 4550
@@
 F 0 "D15" V 9196 5220 50  0000 R CNN
 F 1 "D" V 9105 5220 50  0000 R CNN
-F 2 "Diode_SMD:D_0805_2012Metric_Pad1.15x1.40mm_HandSolder" H 9150 5300 50  0001 C CNN
+F 2 "Diode_SMD:D_0603_1608Metric_Pad1.05x0.95mm_HandSolder" H 9150 5300 50  0001 C CNN
 F 3 "~" H 9150 5300 50  0001 C CNN
 	1    9150 5300
@@
 F 0 "D20" V 9196 5970 50  0000 R CNN
 F 1 "D" V 9105 5970 50  0000 R CNN
-F 2 "Diode_SMD:D_0805_2012Metric_Pad1.15x1.40mm_HandSolder" H 9150 6050 50  0001 C CNN
+F 2 "Diode_SMD:D_0603_1608Metric_Pad1.05x0.95mm_HandSolder" H 9150 6050 50  0001 C CNN
 F 3 "~" H 9150 6050 50  0001 C CNN
 	1    9150 6050
@@
 NoConn ~ 2350 2750
 NoConn ~ 3250 1750
-NoConn ~ 3250 1950
 $Comp
 L power:GND #PWR03
 U 1 1 606B0E12
-P 3950 2050
-F 0 "#PWR03" H 3950 1800 50  0001 C CNN
-F 1 "GND" H 3955 1877 50  0000 C CNN
-F 2 "" H 3950 2050 50  0001 C CNN
-F 3 "" H 3950 2050 50  0001 C CNN
-	1    3950 2050
+P 4850 2050
+F 0 "#PWR03" H 4850 1800 50  0001 C CNN
+F 1 "GND" H 4855 1877 50  0000 C CNN
+F 2 "" H 4850 2050 50  0001 C CNN
+F 3 "" H 4850 2050 50  0001 C CNN
+	1    4850 2050
 	1    0    0    -1
 $EndComp
@@
 $EndComp
 Wire Wire Line
-	3950 1850 3950 2050
+	4850 1850 4850 1950
 Wire Wire Line
 	3750 1650 3750 2050
@@
 Wire Wire Line
 	3750 2050 3250 2050
-Wire Wire Line
-	3250 1850 3950 1850
 Text GLabel 3250 2150 2    50   Input ~ 0
 Col4
@@
 	1    0    0    -1
 $EndComp
+$Comp
+L Switch:SW_Push Reset1
+U 1 1 6066BACD
+P 4350 1950
+F 0 "Reset1" H 4350 2235 50  0000 C CNN
+F 1 "SW_Push" H 4350 2144 50  0000 C CNN
+F 2 "Button_Switch_THT:SW_PUSH_6mm" H 4350 2150 50  0001 C CNN
+F 3 "~" H 4350 2150 50  0001 C CNN
+	1    4350 1950
+	1    0    0    -1
+$EndComp
+Wire Wire Line
+	3250 1950 4150 1950
+Wire Wire Line
+	3250 1850 4850 1850
+Wire Wire Line
+	4550 1950 4850 1950
+Connection ~ 4850 1950
+Wire Wire Line
+	4850 1950 4850 2050
 $EndSCHEMATC

Commit message: v0.2
Parts:
- added D21: LED_RGBC, LED_THT:LED_D5.0mm-4_RGB, symbol Device:LED_RGBC
- added R1, R2, R3: 220Ω, Resistor_THT:R_Axial_DIN0207_L6.3mm_D2.5mm_P10.16mm_Horizontal, symbol Device:R
Connections:
- net labels added: Blue, Green, Red
- wire segments 56 -> 80
- no-connect marks 10 -> 7
Other:
- moved on the sheet: D1, D10, D11, D12, D13, D14, D15, D16, D17, D18, D19, D2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

Commit message: v0.4
Changed lines of the file:
@@
 Sheet 1 1
 Title "CraftPad"
-Date "2021-04-04"
-Rev "V0.3 RGB LED"
+Date "2021-04-05"
+Rev "V0.4 Clean Matrix"
 Comp "James Sa"
 Comment1 ""
@@
 	2350 2050 1400 2050
 Connection ~ 1400 2050
+Text GLabel 3250 2350 2    50   Input ~ 0
+Col1
+Text GLabel 2350 2150 0    50   Input ~ 0
+Row1
+Text GLabel 2350 2350 0    50   Input ~ 0
+Row2
 Text GLabel 2350 2650 0    50   Input ~ 0
-Col1
-Text GLabel 3250 2350 2    50   Input ~ 0
-Row1
-Text GLabel 3250 2450 2    50   Input ~ 0
-Row2
-Text GLabel 3250 2550 2    50   Input ~ 0
 Row3
-Text GLabel 2350 2750 0    50   Input ~ 0
-Row4
 NoConn ~ 2350 1750
 NoConn ~ 2350 1850
-NoConn ~ 2350 2150
+NoConn ~ 3250 2250
 NoConn ~ 2350 2250
-NoConn ~ 2350 2350
 NoConn ~ 3250 2850
+NoConn ~ 3250 2150
 NoConn ~ 3250 1750
 $Comp
@@
 	1    0    0    -1
 $EndComp
+Text GLabel 3250 2550 2    50   Input ~ 0
+Col3
+Text GLabel 3250 2450 2    50   Input ~ 0
+Col2
+Text GLabel 3250 2750 2    50   Input ~ 0
+Col5
+Wire Wire Line
+	3750 2050 3250 2050
 Text GLabel 3250 2650 2    50   Input ~ 0
-Col3
-Text GLabel 3250 2750 2    50   Input ~ 0
-Col2
-Text GLabel 3250 2250 2    50   Input ~ 0
-Col5
-Wire Wire Line
-	3750 2050 3250 2050
-Text GLabel 3250 2150 2    50   Input ~ 0
 Col4
 $Comp
@@
 Wire Wire Line
 	6800 1950 6550 1950
+Text GLabel 2350 2750 0    50   Input ~ 0
+Row4
 $EndSCHEMATC

Commit message: RGBA
Parts:
- removed D21: LED_RGBC, LED_THT:LED_D5.0mm-4_RGB, symbol Device:LED_RGBC
- added D21: LED_RGBA, LED_THT:LED_D5.0mm-4_RGB, symbol Device:LED_RGBA
Connections:
- wire segments 80 -> 81
Other:
- moved on the sheet: R1, R2, R3
Changed lines of the file:
@@
 Wire Wire Line
 	3900 7500 4900 7500
-$Comp
-L Device:LED_RGBC D21
-U 1 1 60742CCE
-P 5850 1950
-F 0 "D21" H 5850 2447 50  0000 C CNN
-F 1 "LED_RGBC" H 5850 2356 50  0000 C CNN
-F 2 "LED_THT:LED_D5.0mm-4_RGB" H 5850 1900 50  0001 C CNN
-F 3 "~" H 5850 1900 50  0001 C CNN
-	1    5850 1950
-	1    0    0    -1
-$EndComp
 Text GLabel 2350 2450 0    50   Input ~ 0
 Blue
-Text GLabel 6800 2150 2    50   Input ~ 0
+Text GLabel 5950 2050 0    50   Input ~ 0
 Blue
 Text GLabel 2350 2550 0    50   Input ~ 0
 Green
-Text GLabel 6800 1950 2    50   Input ~ 0
+Text GLabel 5950 1850 0    50   Input ~ 0
 Green
 Text GLabel 2350 2850 0    50   Input ~ 0
 Red
-Text GLabel 6800 1750 2    50   Input ~ 0
+Text GLabel 5950 1650 0    50   Input ~ 0
 Red
 Wire Wire Line
 	1400 2050 1400 3000
-Wire Wire Line
-	5650 1950 4850 1950
 $Comp
 L Device:R R1
 U 1 1 60780F98
-P 6400 1750
-F 0 "R1" V 6193 1750 50  0000 C CNN
-F 1 "220Ω" V 6284 1750 50  0000 C CNN
-F 2 "Resistor_THT:R_Axial_DIN0207_L6.3mm_D2.5mm_P10.16mm_Horizontal" V 6330 1750 50  0001 C CNN
-F 3 "~" H 6400 1750 50  0001 C CNN
-	1    6400 1750
-	0    1    1    0
+P 6350 1650
+F 0 "R1" V 6143 1650 50  0000 C CNN
+F 1 "220Ω" V 6234 1650 50  0000 C CNN
+F 2 "Resistor_THT:R_Axial_DIN0207_L6.3mm_D2.5mm_P10.16mm_Horizontal" V 6280 1650 50  0001 C CNN
+F 3 "~" H 6350 1650 50  0001 C CNN
+	1    6350 1650
+	0    -1   -1   0
 $EndComp
 Wire Wire Line
-	6050 1750 6250 1750
+	6700 1650 6500 1650
 Wire Wire Line
-	6800 1750 6550 1750
+	5950 1650 6200 1650
 $Comp
 L Device:R R3
 U 1 1 6078ACD2
-P 6400 2150
-F 0 "R3" V 6193 2150 50  0000 C CNN
-F 1 "220Ω" V 6284 2150 50  0000 C CNN
-F 2 "Resistor_THT:R_Axial_DIN0207_L6.3mm_D2.5mm_P10.16mm_Horizontal" V 6330 2150 50  0001 C CNN
-F 3 "~" H 6400 2150 50  0001 C CNN
-	1    6400 2150
-	0    1    1    0
+P 6350 2050
+F 0 "R3" V 6143 2050 50  0000 C CNN
+F 1 "220Ω" V 6234 2050 50  0000 C CNN
+F 2 "Resistor_THT:R_Axial_DIN0207_L6.3mm_D2.5mm_P10.16mm_Horizontal" V 6280 2050 50  0001 C CNN
+F 3 "~" H 6350 2050 50  0001 C CNN
+	1    6350 2050
+	0    -1   -1   0
 $EndComp
 Wire Wire Line
-	6050 2150 6250 2150
+	6700 2050 6500 2050
 Wire Wire Line
-	6800 2150 6550 2150
+	5950 2050 6200 2050
 $Comp
 L Device:R R2
 U 1 1 6079007C
-P 6400 1950
-F 0 "R2" V 6193 1950 50  0000 C CNN
-F 1 "220Ω" V 6284 1950 50  0000 C CNN
-F 2 "Resistor_THT:R_Axial_DIN0207_L6.3mm_D2.5mm_P10.16mm_Horizontal" V 6330 1950 50  0001 C CNN
-F 3 "~" H 6400 1950 50  0001 C CNN
-	1    6400 1950
-	0    1    1    0
+P 6350 1850
+F 0 "R2" V 6143 1850 50  0000 C CNN
+F 1 "220Ω" V 6234 1850 50  0000 C CNN
+F 2 "Resistor_THT:R_Axial_DIN0207_L6.3mm_D2.5mm_P10.16mm_Horizontal" V 6280 1850 50  0001 C CNN
+F 3 "~" H 6350 1850 50  0001 C CNN
+	1    6350 1850
+	0    -1   -1   0
 $EndComp
 Wire Wire Line
-	6050 1950 6250 1950
+	6700 1850 6500 1850
 Wire Wire Line
-	6800 1950 6550 1950
+	5950 1850 6200 1850
 Text GLabel 2350 2750 0    50   Input ~ 0
 Row4
+$Comp
+L Device:LED_RGBA D21
+U 1 1 606B6703
+P 6900 1850
+F 0 "D21" H 6900 2347 50  0000 C CNN
+F 1 "LED_RGBA" H 6900 2256 50  0000 C CNN
+F 2 "LED_THT:LED_D5.0mm-4_RGB" H 6900 1800 50  0001 C CNN
+F 3 "~" H 6900 1800 50  0001 C CNN
+	1    6900 1850
+	1    0    0    -1
+$EndComp
+Wire Wire Line
+	7100 1850 7350 1850
+Wire Wire Line
+	7350 1850 7350 1450
+$Comp
+L power:VCC #PWR0101
+U 1 1 606D791F
+P 7350 1450
+F 0 "#PWR0101" H 7350 1300 50  0001 C CNN
+F 1 "VCC" H 7365 1623 50  0000 C CNN
+F 2 "" H 7350 1450 50  0001 C CNN
+F 3 "" H 7350 1450 50  0001 C CNN
+	1    7350 1450
+	1    0    0    -1
+$EndComp
 $EndSCHEMATC
